File: PCB/interface/interface.sch (KiCad schematic (older format))
At the start: 119 parts, among them J1 24VAC, J10 RS485, J2 Brake, J3 Motor, J4 Limit, J5 LED_G, J6 Ground, J7 LED_B, J8 UART, J9 POT, K1 G2R-1-E, K2 G2R-1-E, K3 G2R-1-E, K4 G2R-1-E, SW1 SW_SPST, U1 DCDC-isolator, U10 PC817, U11 74HCT595, U12 ESP-07, U13 AT24C64, U14 LM358, U15 HCNR201, U16 PC817, U17 LM358, U18 6N137, U19 MAX485E, U2 L7812, U20 6N137, U3 DCDC-isolator, U4 ULN2003A, U5 AMS1117-3.3, U6 PC817, U7 PC817, U8 PC817, U9 PC817

Commit message: first release
Parts:
- R37, R38: value 8K2 -> 18K
Changed lines of the file:
@@
 P 7400 5100
 F 0 "R37" H 7341 5054 50  0000 R CNN
-F 1 "8K2" H 7341 5145 50  0000 R CNN
+F 1 "18K" H 7341 5145 50  0000 R CNN
 F 2 "digikey-footprints:0805" H 7400 5100 50  0001 C CNN
 F 3 "~" H 7400 5100 50  0001 C CNN
@@
 P 7650 5100
 F 0 "R38" H 7591 5054 50  0000 R CNN
-F 1 "8K2" H 7591 5145 50  0000 R CNN
+F 1 "18K" H 7591 5145 50  0000 R CNN
 F 2 "digikey-footprints:0805" H 7650 5100 50  0001 C CNN
 F 3 "~" H 7650 5100 50  0001 C CNN
@@
 Wire Wire Line
 	3850 7100 3900 7100
-Connection ~ 3850 7100
 Wire Wire Line
 	3050 6200 3050 6600

Commit message: optimized map projection algo
Parts:
- U18, U20: symbol MySchLib:6N137 -> interface-rescue:6N137-MySchLib
Changed lines of the file:
@@
 EESchema Schematic File Version 4
 LIBS:interface-cache
-EELAYER 28 0
+EELAYER 30 0
 EELAYER END
 $Descr A4 11693 8268
@@
 $EndComp
 $Comp
-L MySchLib:6N137 U20
+L interface-rescue:6N137-MySchLib U20
 U 1 1 5C109423
 P 3550 7300
@@
 $EndComp
 $Comp
-L MySchLib:6N137 U18
+L interface-rescue:6N137-MySchLib U18
 U 1 1 5C11021E
 P 3600 6450

Commit message: New schemetic and PCB with support of Ethernet LAN connection
Parts:
- R1, R2: value 220 -> 10K
- R41: value 470 -> 1K
- R43: value 220 -> 200
Connections:
- no-connect marks 0 -> 1
Changed lines of the file:
@@
 EESchema Schematic File Version 4
-LIBS:interface-cache
 EELAYER 30 0
 EELAYER END
@@
 U 1 1 5BC990BC
 P 1900 4400
-F 0 "U12" H 1900 5381 50  0000 C CNN
-F 1 "ESP-07" H 1900 5290 50  0000 C CNN
+F 0 "U12" H 1700 5400 50  0000 C CNN
+F 1 "ESP-07" H 1700 5300 50  0000 C CNN
 F 2 "MyPCBLib:ESP-07S" H 1900 4400 50  0001 C CNN
 F 3 "http://wiki.ai-thinker.com/_media/esp8266/esp8266_series_modules_user_manual_v1.1.pdf" H 1550 4500 50  0001 C CNN
@@
 U 1 1 5BCB646B
 P 4750 6450
-F 0 "U19" H 4750 7131 50  0000 C CNN
-F 1 "MAX485E" H 4750 7040 50  0000 C CNN
+F 0 "U19" H 4900 7000 50  0000 C CNN
+F 1 "MAX485E" H 4950 6900 50  0000 C CNN
 F 2 "Housings_SOIC:SOIC-8_3.9x4.9mm_Pitch1.27mm" H 4750 5750 50  0001 C CNN
 F 3 "https://datasheets.maximintegrated.com/en/ds/MAX1487E-MAX491E.pdf" H 4750 6500 50  0001 C CNN
@@
 U 1 1 5BECDDDF
 P 8100 5750
-F 0 "U17" H 8200 5600 50  0000 C CNN
-F 1 "LM358" H 8200 5500 50  0000 C CNN
+F 0 "U17" H 8200 6000 50  0000 C CNN
+F 1 "LM358" H 8200 5900 50  0000 C CNN
 F 2 "Housings_SOIC:SOIC-8_3.9x4.9mm_Pitch1.27mm" H 8100 5750 50  0001 C CNN
 F 3 "http://www.ti.com/lit/ds/symlink/lm2904-n.pdf" H 8100 5750 50  0001 C CNN
@@
 $EndComp
 $Comp
-L Device:R_Small R28
-U 1 1 5BF3402D
-P 9300 4900
-F 0 "R28" V 9200 4900 50  0000 C CNN
-F 1 "1K 1W" V 9400 5000 50  0000 C CNN
-F 2 "Resistors_THT:R_Axial_DIN0411_L9.9mm_D3.6mm_P5.08mm_Vertical" H 9300 4900 50  0001 C CNN
-F 3 "~" H 9300 4900 50  0001 C CNN
-	1    9300 4900
-	-1   0    0    1
-$EndComp
-$Comp
 L power:+24V #PWR04
 U 1 1 5BFF2CF6
@@
 P 5150 1950
 F 0 "R2" H 5209 1996 50  0000 L CNN
-F 1 "220" H 5209 1905 50  0000 L CNN
+F 1 "10K" H 5209 1905 50  0000 L CNN
 F 2 "Resistors_THT:R_Axial_DIN0207_L6.3mm_D2.5mm_P10.16mm_Horizontal" H 5150 1950 50  0001 C CNN
 F 3 "~" H 5150 1950 50  0001 C CNN
@@
 P 5150 1300
 F 0 "R1" H 5209 1346 50  0000 L CNN
-F 1 "220" H 5209 1255 50  0000 L CNN
+F 1 "10K" H 5209 1255 50  0000 L CNN
 F 2 "Resistors_THT:R_Axial_DIN0207_L6.3mm_D2.5mm_P10.16mm_Horizontal" H 5150 1300 50  0001 C CNN
 F 3 "~" H 5150 1300 50  0001 C CNN
@@
 P 3900 6700
 F 0 "R41" H 3959 6746 50  0000 L CNN
-F 1 "470" H 3959 6655 50  0000 L CNN
+F 1 "1K" H 3959 6655 50  0000 L CNN
 F 2 "digikey-footprints:0805" H 3900 6700 50  0001 C CNN
 F 3 "~" H 3900 6700 50  0001 C CNN
@@
 P 3100 7200
 F 0 "R43" V 2904 7200 50  0000 C CNN
-F 1 "220" V 2995 7200 50  0000 C CNN
+F 1 "200" V 2995 7200 50  0000 C CNN
 F 2 "digikey-footprints:0805" H 3100 7200 50  0001 C CNN
 F 3 "~" H 3100 7200 50  0001 C CNN
@@
 Wire Wire Line
 	8900 1550 8900 1600
+NoConn ~ 7200 5800
+$Comp
+L Device:R_Small R28
+U 1 1 5BF3402D
+P 9300 4900
+F 0 "R28" V 9200 4900 50  0000 C CNN
+F 1 "1K 1W" V 9400 5000 50  0000 C CNN
+F 2 "Resistors_THT:R_Axial_DIN0411_L9.9mm_D3.6mm_P5.08mm_Vertical" H 9300 4900 50  0001 C CNN
+F 3 "~" H 9300 4900 50  0001 C CNN
+	1    9300 4900
+	-1   0    0    1
+$EndComp
 $EndSCHEMATC
