File: PCB/interface_SPI_LAN/interface_SPI_LAN.sch (KiCad schematic (older format))
At the start: 129 parts, among them J1 24VAC, J10 LIMIT12, J11 POT, J2 0, J3 JTAG, J4 Power, J5 Control Signals, J6 HR913550A, J7 Sensor Feedback, J8 UART, J9 POT, Q1 8550, Q2 TIP127, Q3 MMBT5551, SW1 SW_SPST, SW2 CW, SW3 CCW, SW4 SET, U1 B1205-1W, U10 EL357, U11 74HCT595, U12 EL357, U13 AT24C64, U14 LM358, U15 HCNR201, U17 LMV358, U2 ESP32-WROOM-32, U3 LM317_TO-220, U4 L78L05_SOT89, U5 AMS1117-3.3, U6 OLED_128x32_4pin, U9 HCNR201

Commit message: Implenting SPWM
Parts:
- removed C15, C41: 104, lc_lib:0805_C, symbol Device:C_Small
- removed R24, R25: 4.7K, lc_lib:0805_R, symbol Device:R_Small
- removed R33, R42: 10, lc_lib:0805_R, symbol Device:R_Small
- removed U13: AT24C64, lc_lib:SOIC-8_150MIL, symbol Memory_NVRAM:FM24C64B
- added C?: 1uF, lc_lib:0805_C, symbol Device:C_Small
- added J?: UART_EXT, Connector_PinHeader_2.54mm:PinHeader_1x04_P2.54mm_Vertical, symbol Connector_Generic:Conn_01x04
- added R? (x3): 100, lc_lib:0805_R, symbol Device:R_Small
- added R? (x5): 10, lc_lib:0805_R, symbol Device:R_Small
- C39, C40: value 104 -> 10nF
- R17: value 4.7K -> 1K
Connections:
- net labels added: 485RW, BOOT_OE, BOOT_TX_EXT, ETH_CSX, ETH_INTX, ETH_MISO, ETH_MOSI, ETH_RSTX, ETH_SCK, INTX, IO_INTX, ISense2, LEDAX, LMTX2_TDO, RX_EXT, SPWM3, TCK, TMS, TX_EXT, VSPI_MISO, VSPI_MOSI, VSPI_SCK
- net labels removed: BOOT_WP, LEDAX_485RW, OE
- wire segments 525 -> 531
- no-connect marks 7 -> 6
Other:
- note removed: "BOOT2 PD"
- note removed: "EEPROM I2C ADDR: 0x00"
- note removed: "High for CLKin"
- note removed: "REGOFF=0: Use Internal 1.2V"
- note removed: "nINTSEL=1 REFCLK in"
- moved on the sheet: C13, C23, C?, D11, D12, J6, R17, R35, R36, R38, R39, R4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
