File: PCB/motor_control_SPWM/H.sch (KiCad schematic (older format))
At the start: 16 parts, among them Q6 IRFS4310Z, Q7 IRFS4310Z, Q8 IRFS4310Z, Q9 IRFS4310Z

Commit message: Implenting SPWM
Changed lines of the file:
@@
 AR Path="/63B00E4C/63A5E297" Ref="Q?"  Part="1"
 AR Path="/63B13A24/63A5E297" Ref="Q10"  Part="1"
-F 0 "Q6" H 4200 2800 50  0000 L CNN
+F 0 "Q10" H 4200 2800 50  0000 L CNN
 F 1 "IRFS4310Z" H 3900 2700 50  0000 L CNN
 F 2 "lc_lib:TO-252-2" H 4550 2525 50  0001 L CIN
@@
 AR Path="/63B00E4C/63A5E29D" Ref="Q?"  Part="1"
 AR Path="/63B13A24/63A5E29D" Ref="Q11"  Part="1"
-F 0 "Q7" H 4554 3746 50  0000 L CNN
+F 0 "Q11" H 4554 3746 50  0000 L CNN
 F 1 "IRFS4310Z" H 3950 3850 50  0000 L CNN
 F 2 "lc_lib:TO-252-2" H 4550 3625 50  0001 L CIN
@@
 AR Path="/63B00E4C/63A5E2A3" Ref="Q?"  Part="1"
 AR Path="/63B13A24/63A5E2A3" Ref="Q13"  Part="1"
-F 0 "Q9" H 5954 3746 50  0000 L CNN
+F 0 "Q13" H 5954 3746 50  0000 L CNN
 F 1 "IRFS4310Z" H 5400 3850 50  0000 L CNN
 F 2 "lc_lib:TO-252-2" H 5950 3625 50  0001 L CIN
@@
 AR Path="/63B00E4C/63A5E2A9" Ref="Q?"  Part="1"
 AR Path="/63B13A24/63A5E2A9" Ref="Q12"  Part="1"
-F 0 "Q8" H 5954 2646 50  0000 L CNN
+F 0 "Q12" H 5954 2646 50  0000 L CNN
 F 1 "IRFS4310Z" H 5950 2550 50  0000 L CNN
 F 2 "lc_lib:TO-252-2" H 5950 2525 50  0001 L CIN
@@
 AR Path="/63B00E4C/63A66C07" Ref="D?"  Part="1"
 AR Path="/63B13A24/63A66C07" Ref="D10"  Part="1"
-F 0 "D6" H 3600 2666 50  0000 C CNN
+F 0 "D10" H 3600 2666 50  0000 C CNN
 F 1 "4148" H 3600 2575 50  0000 C CNN
 F 2 "MyPCBLib:SOD-123" H 3600 2450 50  0001 C CNN
@@
 AR Path="/63B00E4C/63A67731" Ref="R?"  Part="1"
 AR Path="/63B13A24/63A67731" Ref="R50"  Part="1"
-F 0 "R34" V 3400 2600 50  0000 C CNN
+F 0 "R50" V 3400 2600 50  0000 C CNN
 F 1 "10" V 3500 2600 50  0000 C CNN
 F 2 "lc_lib:0805_R" H 3600 2600 50  0001 C CNN
@@
 AR Path="/63B00E4C/63A6B27E" Ref="D?"  Part="1"
 AR Path="/63B13A24/63A6B27E" Ref="D11"  Part="1"
-F 0 "D7" H 3600 3766 50  0000 C CNN
+F 0 "D11" H 3600 3766 50  0000 C CNN
 F 1 "4148" H 3600 3675 50  0000 C CNN
 F 2 "MyPCBLib:SOD-123" H 3600 3550 50  0001 C CNN
@@
 AR Path="/63B00E4C/63A6B284" Ref="R?"  Part="1"
 AR Path="/63B13A24/63A6B284" Ref="R51"  Part="1"
-F 0 "R35" V 3400 3700 50  0000 C CNN
+F 0 "R51" V 3400 3700 50  0000 C CNN
 F 1 "10" V 3500 3700 50  0000 C CNN
 F 2 "lc_lib:0805_R" H 3600 3700 50  0001 C CNN
@@
 AR Path="/63B00E4C/63A6D9D4" Ref="D?"  Part="1"
 AR Path="/63B13A24/63A6D9D4" Ref="D12"  Part="1"
-F 0 "D8" H 6500 2666 50  0000 C CNN
+F 0 "D12" H 6500 2666 50  0000 C CNN
 F 1 "4148" H 6500 2575 50  0000 C CNN
 F 2 "MyPCBLib:SOD-123" H 6500 2450 50  0001 C CNN
@@
 AR Path="/63B00E4C/63A6D9DA" Ref="R?"  Part="1"
 AR Path="/63B13A24/63A6D9DA" Ref="R56"  Part="1"
-F 0 "R40" V 6300 2600 50  0000 C CNN
+F 0 "R56" V 6300 2600 50  0000 C CNN
 F 1 "10" V 6400 2600 50  0000 C CNN
 F 2 "lc_lib:0805_R" H 6500 2600 50  0001 C CNN
@@
 AR Path="/63B00E4C/63A6EE71" Ref="D?"  Part="1"
 AR Path="/63B13A24/63A6EE71" Ref="D13"  Part="1"
-F 0 "D9" H 6500 3766 50  0000 C CNN
+F 0 "D13" H 6500 3766 50  0000 C CNN
 F 1 "4148" H 6500 3675 50  0000 C CNN
 F 2 "MyPCBLib:SOD-123" H 6500 3550 50  0001 C CNN
@@
 AR Path="/63B00E4C/63A6EE77" Ref="R?"  Part="1"
 AR Path="/63B13A24/63A6EE77" Ref="R57"  Part="1"
-F 0 "R41" V 6300 3700 50  0000 C CNN
+F 0 "R57" V 6300 3700 50  0000 C CNN
 F 1 "10" V 6400 3700 50  0000 C CNN
 F 2 "lc_lib:0805_R" H 6500 3700 50  0001 C CNN
@@
 AR Path="/63B00E4C/63A6FE13" Ref="R?"  Part="1"
 AR Path="/63B13A24/63A6FE13" Ref="R52"  Part="1"
-F 0 "R36" V 3900 2800 50  0000 C CNN
+F 0 "R52" V 3900 2800 50  0000 C CNN
 F 1 "100K" V 4000 2800 50  0000 C CNN
 F 2 "lc_lib:0805_R" H 4100 2800 50  0001 C CNN
@@
 AR Path="/63B00E4C/63A71E87" Ref="R?"  Part="1"
 AR Path="/63B13A24/63A71E87" Ref="R53"  Part="1"
-F 0 "R37" V 3950 3950 50  0000 C CNN
+F 0 "R53" V 3950 3950 50  0000 C CNN
 F 1 "100K" V 4050 3950 50  0000 C CNN
 F 2 "lc_lib:0805_R" H 4150 3950 50  0001 C CNN
@@
 AR Path="/63B00E4C/63A748CC" Ref="R?"  Part="1"
 AR Path="/63B13A24/63A748CC" Ref="R54"  Part="1"
-F 0 "R38" V 5700 2800 50  0000 C CNN
+F 0 "R54" V 5700 2800 50  0000 C CNN
 F 1 "100K" V 5800 2800 50  0000 C CNN
 F 2 "lc_lib:0805_R" H 5900 2800 50  0001 C CNN
@@
 AR Path="/63B00E4C/63A75C61" Ref="R?"  Part="1"
 AR Path="/63B13A24/63A75C61" Ref="R55"  Part="1"
-F 0 "R39" V 5700 3950 50  0000 C CNN
+F 0 "R55" V 5700 3950 50  0000 C CNN
 F 1 "100K" V 5800 3950 50  0000 C CNN
 F 2 "lc_lib:0805_R" H 5900 3950 50  0001 C CNN
