File: PCB/motor_control_SPWM/file63C26554.sch (KiCad schematic (older format))
At the start: 15 parts, among them U16 LM324

Commit message: Implenting SPWM
Parts:
- added R22, R23, R24, R25: 1K, lc_lib:0805_R, symbol Device:R_Small
Connections:
- net GNDS: now also R24.1, R25.1
- net VISense1: now also R22.2; no longer U16.5 (+)
- net VISense2: now also R23.2; no longer U16.10 (+)
- new net: R22.1, R24.2, U16.5 (+)
- new net: R23.1, R25.2, U16.10 (+)
Other:
- moved on the sheet: TP8
Changed lines of the file:
@@
 	4950 2500 4850 2500
 Wire Wire Line
-	2950 4200 3400 4200
+	2950 4200 3050 4200
 Wire Wire Line
 	2950 5300 3400 5300
@@
 L Connector:TestPoint TP8
 U 1 1 64BC7BC4
-P 3400 4100
-F 0 "TP8" H 3458 4218 50  0000 L CNN
-F 1 "VIS1" H 3458 4127 50  0000 L CNN
-F 2 "TestPoint:TestPoint_Pad_D1.0mm" H 3600 4100 50  0001 C CNN
-F 3 "~" H 3600 4100 50  0001 C CNN
-	1    3400 4100
-	1    0    0    -1
-$EndComp
-Wire Wire Line
-	3400 4100 3400 4200
-Connection ~ 3400 4200
-Wire Wire Line
-	3400 4200 4250 4200
+P 3050 4100
+F 0 "TP8" H 3108 4218 50  0000 L CNN
+F 1 "VIS1" H 3108 4127 50  0000 L CNN
+F 2 "TestPoint:TestPoint_Pad_D1.0mm" H 3250 4100 50  0001 C CNN
+F 3 "~" H 3250 4100 50  0001 C CNN
+	1    3050 4100
+	1    0    0    -1
+$EndComp
+Wire Wire Line
+	3050 4100 3050 4200
 $Comp
 L Connector:TestPoint TP9
@@
 Connection ~ 3400 5300
 Wire Wire Line
-	3400 5300 4250 5300
+	3400 5300 3600 5300
+Connection ~ 3050 4200
+Wire Wire Line
+	3050 4200 3600 4200
+$Comp
+L Device:R_Small R22
+U 1 1 638CAB19
+P 3700 4200
+F 0 "R22" V 3800 4100 50  0000 C CNN
+F 1 "1K" V 3800 4250 50  0000 C CNN
+F 2 "lc_lib:0805_R" H 3700 4200 50  0001 C CNN
+F 3 "~" H 3700 4200 50  0001 C CNN
+	1    3700 4200
+	0    1    1    0
+$EndComp
+Wire Wire Line
+	3800 4200 4000 4200
+$Comp
+L Device:R_Small R24
+U 1 1 638CB355
+P 4000 4000
+F 0 "R24" V 3900 4150 50  0000 C CNN
+F 1 "1K" V 3900 4000 50  0000 C CNN
+F 2 "lc_lib:0805_R" H 4000 4000 50  0001 C CNN
+F 3 "~" H 4000 4000 50  0001 C CNN
+	1    4000 4000
+	1    0    0    -1
+$EndComp
+Wire Wire Line
+	4000 4100 4000 4200
+Connection ~ 4000 4200
+Wire Wire Line
+	4000 4200 4250 4200
+$Comp
+L power:GNDS #PWR0109
+U 1 1 638CCC50
+P 4150 3900
+F 0 "#PWR0109" H 4150 3650 50  0001 C CNN
+F 1 "GNDS" H 4155 3727 50  0000 C CNN
+F 2 "" H 4150 3900 50  0001 C CNN
+F 3 "" H 4150 3900 50  0001 C CNN
+	1    4150 3900
+	1    0    0    -1
+$EndComp
+Wire Wire Line
+	4150 3900 4150 3850
+Wire Wire Line
+	4150 3850 4000 3850
+Wire Wire Line
+	4000 3850 4000 3900
+$Comp
+L Device:R_Small R23
+U 1 1 638CE2EE
+P 3700 5300
+F 0 "R23" V 3600 5450 50  0000 C CNN
+F 1 "1K" V 3600 5300 50  0000 C CNN
+F 2 "lc_lib:0805_R" H 3700 5300 50  0001 C CNN
+F 3 "~" H 3700 5300 50  0001 C CNN
+	1    3700 5300
+	0    1    1    0
+$EndComp
+Wire Wire Line
+	3800 5300 4050 5300
+$Comp
+L Device:R_Small R25
+U 1 1 638CE819
+P 4050 5200
+F 0 "R25" V 3950 5350 50  0000 C CNN
+F 1 "1K" V 3950 5200 50  0000 C CNN
+F 2 "lc_lib:0805_R" H 4050 5200 50  0001 C CNN
+F 3 "~" H 4050 5200 50  0001 C CNN
+	1    4050 5200
+	1    0    0    -1
+$EndComp
+Connection ~ 4050 5300
+Wire Wire Line
+	4050 5300 4250 5300
+$Comp
+L power:GNDS #PWR0110
+U 1 1 638CECC0
+P 4200 5000
+F 0 "#PWR0110" H 4200 4750 50  0001 C CNN
+F 1 "GNDS" H 4205 4827 50  0000 C CNN
+F 2 "" H 4200 5000 50  0001 C CNN
+F 3 "" H 4200 5000 50  0001 C CNN
+	1    4200 5000
+	1    0    0    -1
+$EndComp
+Wire Wire Line
+	4200 5000 4050 5000
+Wire Wire Line
+	4050 5000 4050 5100
 $EndSCHEMATC
