File: PCB/motor_control_SPWM/motor_control.kicad_pcb (KiCad board)
At the start: 2 copper layers, 100 x 75 mm, 134 parts, among them J1 Sensor Feedback, J2 Control Signals, J3 Power, J4 MOT1, J5 MOT2, J6 Ground, J7 DC in, K1 G2RL-1-E, Q1 8050, Q10 IRFS4310Z, Q11 IRFS4310Z, Q12 IRFS4310Z, Q13 IRFS4310Z, Q6 IRFS4310Z, Q7 IRFS4310Z, Q8 IRFS4310Z, Q9 IRFS4310Z, U1 LTV-357T, U10 IR2104, U11 IR2104, U12 IR2104, U13 CC6902-10A, U14 CC6902-10A, U15 74HC00, U16 LM324, U17 74HC04, U18 L78L05_SOT89, U2 LTV-357T, U3 LTV-357T, U4 LTV-357T, U5 LTV-357T, U6 LTV-357T, U7 LTV-357T, U8 LTV-357T, U9 IR2104

Commit message: Implenting SPWM
Parts:
- added R22: 1K, lc_lib:0805_R, F.Cu at (42.8, 35.5)
- added R23: 1K, lc_lib:0805_R, F.Cu at (59.6, 31.5)
- added R24: 1K, lc_lib:0805_R, F.Cu at (40.2, 35.5)
- added R25: 1K, lc_lib:0805_R, F.Cu at (40.2, 23.0)
- added R28: 0, lc_lib:1206_R, F.Cu at (85.2, 30.2)
- added R29: 47K, lc_lib:0805_R, F.Cu at (100.0, 87.5)
- added SC3: M3, MyPCBLib:M3_Screwhole, F.Cu at (70.0, 24.0)
- added SC4: M3, MyPCBLib:M3_Screwhole, F.Cu at (96.5, 52.0)
- R17: value 10 -> 10K
- moved TP8 17.8 mm to (55.5, 69.8)
- moved C17 12.3 mm to (32.0, 26.0), turned to 90 degrees
- moved C18 5.00 mm to (37.5, 35.5)
- moved TP9 3.25 mm to (55.5, 33.5)
- moved R47 3.00 mm to (36.8, 23.0), turned to 270 degrees
- moved D5 2.25 mm to (105.2, 93.2)
- moved R45 2.15 mm to (34.8, 35.5)
- moved C1 1.50 mm to (29.5, 26.0), turned to 90 degrees
- moved TP10 1.50 mm to (22.8, 30.0)
- moved TP11 1.50 mm to (22.8, 32.5)
- moved R56 0.60 mm to (56.6, 46.0)
- moved R42 0.29 mm to (34.6, 27.0)
Connections:
- J3 pad 2: +VDC -> /+VDC_Out
- J3 pad 4: +VDC -> /+VDC_Out
- J3 pad 6: +VDC -> /+VDC_Out
- J3 pad 8: +VDC -> /+VDC_Out
- U16 pad 10: /VIOut2 -> Net-(R23-Pad1)
- U16 pad 5: /VIOut1 -> Net-(R22-Pad1)
Routing:
- net Net-(R23-Pad1): track 0.00 -> 24.5 mm, vias 0 -> 2
- net /VIOut2: track 32.6 -> 14.1 mm, vias 2 -> 1
- net +5VISO: track 120.5 -> 129.4 mm, vias 11 -> 10
- net GNDS: track 122.4 -> 130.7 mm, vias 34 -> 32
- net Net-(Q1-Pad1): track 2.75 -> 9.80 mm
- net Net-(R47-Pad1): track 6.03 -> 12.0 mm
- net Net-(R22-Pad1): track 0.00 -> 5.27 mm
- net /RELIN2: track 45.3 -> 40.6 mm
- net GNDPWR: track 41.7 -> 37.2 mm, vias 87 -> 88
- net /VIOut1: track 72.4 -> 69.9 mm
- net /RELIN3: track 35.5 -> 33.7 mm
- net /CurrentSensing/VMID: track 19.0 -> 17.5 mm, vias 1 -> 2
- net /RELIN5: track 33.3 -> 32.1 mm
- net Net-(D5-Pad2): track 6.78 -> 7.71 mm
- net /MOT2_N: track 91.5 -> 92.2 mm
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- added copper zone on F.Cu, net /+VDC_Out
- removed copper zone on B.Cu, net (none)
Other:
- board text added: "+"
- board text added: "+12V"
- board text added: "+5V"
- board text added: "-"
- board text added: "CCW"
- board text added: "COM"
- board text added: "CW"
- board text added: "GND"
- board text added: "Power to Control Board"
- board text added: "SPWM Motor Control Board V0.1 By Zening, Lu (BI4WOP) Nov 30, 2022"
- board text added: "VMain"
- board text added: "Vmain"
