File: PCB/motor_control_SPWM/motor_control.sch (KiCad schematic (older format))
At the start: 40 parts

Commit message: motor control board with SPWM support`
Parts:
- removed C?: 104, lc_lib:0805_C, symbol Device:C_Small
- removed J?: TRIAC_AUX1, Connector_Phoenix_MSTB:PhoenixContact_MSTBA_2,5_3-G-5,08_1x03_P5.08mm_Horizontal, symbol Connector:Screw_Terminal_01x02
- removed J?: MOT2, Connector_Phoenix_MSTB:PhoenixContact_MSTBA_2,5_3-G-5,08_1x03_P5.08mm_Horizontal, symbol Connector:Screw_Terminal_01x03
- removed K? (x3): G2RL-1-E, symbol MySchLib:G2RL-1-E
- removed Q? (x4): IRFS4310Z, Package_TO_SOT_SMD:TO-263-2, symbol Transistor_FET:IRFS4310Z
- removed R? (x2): 100, symbol Device:R_Small
- removed R? (x2): 10K, symbol Device:R_Small
- removed R?: 100, lc_lib:0805_R, symbol Device:R_Small
- removed U?: ACS712xLCTR-30A, Package_SO:SOIC-8_3.9x4.9mm_P1.27mm, symbol Sensor_Current:ACS712xLCTR-30A
- added C1: 10uF, lc_lib:0805_C, symbol Device:C_Small
- added C10, C11, C12, C14: 104, lc_lib:0805_C, symbol Device:C_Small
- added C13, C15: 100uF 50V, Capacitor_SMD:CP_Elec_8x10.5, symbol Device:CP_Small
- added C19, C4, C5, C6, C8: 10uF, lc_lib:1206_C, symbol Device:C_Small
- added C2, C21, C22, C3, C7, C9: 1uF, lc_lib:0805_C, symbol Device:C_Small
- added D1, D2, D3, D4: SD103, MyPCBLib:SOD-123, symbol MySchLib:D_Schottky_Small
- added D5: 4148, MyPCBLib:SOD-123, symbol Diode:1N4148
- added J5: MOT2, Connector_Phoenix_MSTB:PhoenixContact_MSTBA_2,5_2-G-5,08_1x02_P5.08mm_Horizontal, symbol Connector:Screw_Terminal_01x02
- added Q1: 8050, lc_lib:SOT-23(SOT-23-3), symbol MySchLib:8050
- added R10, R14, R6, R7, R8, R9: 4.7K, lc_lib:0805_R, symbol Device:R_Small
- added R11, R5: 220, lc_lib:0805_R, symbol Device:R_Small
- added R17: 10, lc_lib:0805_R, symbol Device:R_Small
- added R18, R19: 100, lc_lib:0805_R, symbol Device:R_Small
- added SC1, SC2: M3, MyPCBLib:M3_Screwhole, symbol Connector_Generic:Conn_01x01
- added TP2: H1INL, TestPoint:TestPoint_Pad_D1.0mm, symbol Connector:TestPoint
- added TP3: H1INR, TestPoint:TestPoint_Pad_D1.0mm, symbol Connector:TestPoint
- added TP4: H2INL, TestPoint:TestPoint_Pad_D1.0mm, symbol Connector:TestPoint
- added TP5: H2INR, TestPoint:TestPoint_Pad_D1.0mm, symbol Connector:TestPoint
- added TP6, TP7: GNDP, TestPoint:TestPoint_Pad_D1.0mm, symbol Connector:TestPoint
- added U10, U12: IR2104, lc_lib:SOIC-8_150MIL, symbol Driver_FET:IR2104
- added U13, U14: CC6902-10A, Package_SO:SOIC-8_3.9x4.9mm_P1.27mm, symbol Sensor_Current:ACS712xLCTR-20A
- added U18: L78L05_SOT89, lc_lib:SOT-89(SOT-89-3), symbol Regulator_Linear:L78L05_SOT89
- added U5, U6: LTV-357T, Package_SO:SO-4_4.4x3.6mm_P2.54mm, symbol Isolator:LTV-357T
- J1, J2, J3: renamed from J?; footprint Connector_PinHeader_2.54mm:PinHeader_2x05_P2.54mm_Vertical -> Connector_PinHeader_2.54mm:PinHeader_2x05_P2.54mm_Vertical_SMD
- J6: renamed from J?; footprint Connector_Phoenix_MSTB:PhoenixContact_MSTBA_2,5_3-G-5,08_1x03_P5.08mm_Horizontal -> Connector_Phoenix_MSTB:PhoenixContact_MSTBA_2,5_2-G-5,08_1x02_P5.08mm_Horizontal
- K1: renamed from K?; footprint (none) -> MyPCBLib:G2RL-1-E
- R1, R12, R13, R15, R16, R2, R3, R4: renamed from R?; footprint (none) -> lc_lib:0805_R
- U11, U9: renamed from U?; footprint (none) -> lc_lib:SOIC-8_150MIL
- gave numbers to parts that had none: 9
Connections:
- net labels added: +3.3VISO, +5VISO, BRAKE, DIRREL1, H1LO, H1RO, H1SELL, H1SELR, H2SELL, H2SELR, MOT1_CCW, MOT1_COM, MOT1_CW, MOT2_N, MOT2_P, SDX, SPWM1_OUT, SPWM2_OUT, VIOut1, VIOut2, VISenseOut1, VISenseOut2
- net labels removed: +3.3V, ISense1, Isense, P_metered
- wire segments 139 -> 322
Other:
- note added: "Non Isolated"
- moved on the sheet: F1, J1, J2, J3, J7, K1, R1, R12, R13, R15, R16, R2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

Commit message: Implenting SPWM
Parts:
- added R28: 0, lc_lib:1206_R, symbol Device:R_Small
- added R29: 47K, lc_lib:0805_R, symbol Device:R_Small
- added SC3, SC4: M3, MyPCBLib:M3_Screwhole, symbol Connector_Generic:Conn_01x01
- R17: value 10 -> 10K
Connections:
- net +VDC: now also R28.2; no longer J3.2 (Pin_2), J3.4 (Pin_4), J3.6 (Pin_6), J3.8 (Pin_8)
- net GNDPWR: now also C19.2, R29.2
- net GNDS: no longer C19.2
- net at Q1.1 (B), R17.2: now also R29.1
- new net +VDC_Out: J3.2 (Pin_2), J3.4 (Pin_4), J3.6 (Pin_6), J3.8 (Pin_8), R28.1
Changed lines of the file:
@@
 Wire Wire Line
 	3000 1050 3200 1050
-Connection ~ 3200 1050
 Wire Wire Line
 	3200 1050 3200 1150
@@
 L power:+VDC #PWR021
 U 1 1 62775896
-P 3200 1050
-F 0 "#PWR021" H 3200 950 50  0001 C CNN
-F 1 "+VDC" H 3000 1150 50  0000 C CNN
-F 2 "" H 3200 1050 50  0001 C CNN
-F 3 "" H 3200 1050 50  0001 C CNN
-	1    3200 1050
+P 3200 850
+F 0 "#PWR021" H 3200 750 50  0001 C CNN
+F 1 "+VDC" H 3000 950 50  0000 C CNN
+F 2 "" H 3200 850 50  0001 C CNN
+F 3 "" H 3200 850 50  0001 C CNN
+	1    3200 850
 	1    0    0    -1
 $EndComp
@@
 Wire Wire Line
 	3400 6150 3400 7050
-Text GLabel 1850 2350 2    50   Output ~ 0
+Text GLabel 2500 2350 2    50   Output ~ 0
 +3.3VISO
 Wire Wire Line
@@
 	8050 5050 8050 5300
 Wire Wire Line
-	1800 2350 1850 2350
+	1800 2350 2500 2350
 $Sheet
 S 6900 4800 800  800
@@
 U 1 1 643B21D3
 P 7400 3500
-F 0 "R17" V 7500 3600 50  0000 R CNN
-F 1 "10" V 7500 3500 50  0000 R CNN
+F 0 "R17" V 7500 3650 50  0000 R CNN
+F 1 "10K" V 7500 3500 50  0000 R CNN
 F 2 "lc_lib:0805_R" H 7400 3500 50  0001 C CNN
 F 3 "~" H 7400 3500 50  0001 C CNN
@@
 L power:GNDPWR #PWR036
 U 1 1 643C8B36
-P 7850 3800
-F 0 "#PWR036" H 7850 3600 50  0001 C CNN
-F 1 "GNDPWR" H 7750 3650 50  0000 C CNN
-F 2 "" H 7850 3750 50  0001 C CNN
-F 3 "" H 7850 3750 50  0001 C CNN
-	1    7850 3800
-	1    0    0    -1
-$EndComp
-Wire Wire Line
-	7850 3800 7850 3700
+P 7850 3850
+F 0 "#PWR036" H 7850 3650 50  0001 C CNN
+F 1 "GNDPWR" H 8050 3800 50  0000 C CNN
+F 2 "" H 7850 3800 50  0001 C CNN
+F 3 "" H 7850 3800 50  0001 C CNN
+	1    7850 3850
+	1    0    0    -1
+$EndComp
+Wire Wire Line
+	7850 3850 7850 3800
 $Comp
 L Diode:1N4148 D5
@@
 	1    0    0    -1
 $EndComp
-$Comp
-L power:GNDS #PWR0101
-U 1 1 64657A8A
-P 8900 3700
-F 0 "#PWR0101" H 8900 3450 50  0001 C CNN
-F 1 "GNDS" H 8905 3527 50  0000 C CNN
-F 2 "" H 8900 3700 50  0001 C CNN
-F 3 "" H 8900 3700 50  0001 C CNN
-	1    8900 3700
-	1    0    0    -1
-$EndComp
-Wire Wire Line
-	8900 3700 8900 3550
 Wire Wire Line
 	8900 3350 8900 3200
@@
 Wire Wire Line
 	10500 1200 10500 600
-Wire Wire Line
-	3600 6150 3400 6150
-Connection ~ 3400 6150
 $Comp
 L Regulator_Linear:L78L05_SOT89 U18
@@
 	7850 5550 7850 5950
 Connection ~ 7850 5550
+$Comp
+L power:GNDPWR #PWR0101
+U 1 1 64FEEFDB
+P 8900 3800
+F 0 "#PWR0101" H 8900 3600 50  0001 C CNN
+F 1 "GNDPWR" H 8800 3650 50  0000 C CNN
+F 2 "" H 8900 3750 50  0001 C CNN
+F 3 "" H 8900 3750 50  0001 C CNN
+	1    8900 3800
+	1    0    0    -1
+$EndComp
+Wire Wire Line
+	8900 3550 8900 3800
+$Comp
+L Device:R_Small R28
+U 1 1 63A42B41
+P 3200 950
+F 0 "R28" V 3300 950 50  0000 C CNN
+F 1 "0" V 3300 850 50  0000 C CNN
+F 2 "lc_lib:1206_R" H 3200 950 50  0001 C CNN
+F 3 "~" H 3200 950 50  0001 C CNN
+	1    3200 950
+	-1   0    0    1
+$EndComp
+Connection ~ 3200 1050
+Text Label 3000 1250 0    50   ~ 0
++VDC_Out
+$Comp
+L Connector_Generic:Conn_01x01 SC3
+U 1 1 63A6EA99
+P 10050 5150
+F 0 "SC3" H 10130 5192 50  0000 L CNN
+F 1 "M3" H 10130 5101 50  0000 L CNN
+F 2 "MyPCBLib:M3_Screwhole" H 10050 5150 50  0001 C CNN
+F 3 "~" H 10050 5150 50  0001 C CNN
+	1    10050 5150
+	1    0    0    -1
+$EndComp
+$Comp
+L Connector_Generic:Conn_01x01 SC4
+U 1 1 63A6EA9F
+P 10050 5500
+F 0 "SC4" H 10130 5542 50  0000 L CNN
+F 1 "M3" H 10130 5451 50  0000 L CNN
+F 2 "MyPCBLib:M3_Screwhole" H 10050 5500 50  0001 C CNN
+F 3 "~" H 10050 5500 50  0001 C CNN
+	1    10050 5500
+	1    0    0    -1
+$EndComp
+$Comp
+L Device:R_Small R29
+U 1 1 63AD66DB
+P 7550 3700
+F 0 "R29" V 7450 3600 50  0000 R CNN
+F 1 "47K" V 7450 3800 50  0000 R CNN
+F 2 "lc_lib:0805_R" H 7550 3700 50  0001 C CNN
+F 3 "~" H 7550 3700 50  0001 C CNN
+	1    7550 3700
+	1    0    0    -1
+$EndComp
+Wire Wire Line
+	7550 3600 7550 3500
+Connection ~ 7550 3500
+Wire Wire Line
+	7550 3800 7850 3800
+Connection ~ 7850 3800
+Wire Wire Line
+	7850 3800 7850 3700
 $EndSCHEMATC
